File: 4020 ADSR/4020 ADSR.sch (KiCad schematic (older format))
At the start: 58 parts, among them J1 TRIGGER INPUT, J10 DECAY/SUSTAIN, J11 RELEASE, J2 GATE INPUT, J3 NEGATIVE SUPPLY, J4 GROUND, J5 POSITIVE SUPPLY, J6 ADSR OUTPUT, J7 GROUND, J8 ATTACK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

Commit message: Fix some transistors pinouts
Parts:
- Q3: symbol Device:Q_NJFET_DGS -> Device:Q_NJFET_SGD
- Q6: symbol Device:Q_PNP_ECB -> Device:Q_PNP_EBC
Connections:
- net at A1.3 (+), C1.2, C2.2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: now also Q3.1 (S); no longer Q3.3 (S)
- net at CR6.2 (A), CR7.2 (A), CR8.2 (A)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: now also Q6.3 (C); no longer Q6.2 (C)
- net at J11.1 (Pin_1), R6.1: now also Q3.3 (D); no longer Q3.1 (D)
- net at C5.2, R15.2, R16.1: now also Q6.2 (B); no longer Q6.3 (B)
Changed lines of the file:
@@
 $EndComp
 $Comp
-L Device:Q_NJFET_DGS Q3
+L Device:Q_NJFET_SGD Q3
 U 1 1 6078872B
 P 4400 3250
@@
 $EndComp
 $Comp
-L Device:Q_PNP_ECB Q6
+L Device:Q_PNP_EBC Q6
 U 1 1 6078B4A2
 P 9250 2650

Commit message: various fixes
Changed lines of the file:
@@
 Wire Wire Line
 	8850 4250 8850 4400
+$Comp
+L power:PWR_FLAG #FLG?
+U 1 1 60B5A4D0
+P 1500 6350
+F 0 "#FLG?" H 1500 6425 50  0001 C CNN
+F 1 "PWR_FLAG" H 1400 6500 50  0000 L CNN
+F 2 "" H 1500 6350 50  0001 C CNN
+F 3 "~" H 1500 6350 50  0001 C CNN
+	1    1500 6350
+	1    0    0    -1
+$EndComp
 $EndSCHEMATC
