File: 4014 Ring Modulator/4014 Ring Modulator.sch (KiCad schematic (older format))
At the start: 54 parts, among them J10 NEG. NULL, J18 POS. NULL, J2 Y INPUT, J3 X INPUT, J5 OUTPUT, J6 POSITIVE SUPPLY, J7 GROUND, J8 NEGATIVE SUPPLY, J9 GAIN TRIM, Q1 2N3906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

Commit message: fix J3 vs J4 typo
Parts:
- renumbered J3 to J4
Changed lines of the file:
@@
 Connection ~ 2000 1600
 $Comp
-L Connector_Generic:Conn_01x01 J3
+L Connector_Generic:Conn_01x01 J4
 U 1 1 600D6FF4
 P 950 3150
-F 0 "J3" H 868 2925 50  0000 C CNN
+F 0 "J4" H 868 2925 50  0000 C CNN
 F 1 "X INPUT" H 868 3016 50  0000 C CNN
 F 2 "" H 950 3150 50  0001 C CNN
