File: Board 5/Board 5.sch (KiCad schematic (older format))
At the start: 67 parts, among them J51-20 S/H LEVEL

Commit message: Board 5 fix
Other:
- note added: "LAG OUT"
Changed lines of the file:
@@
 Text Notes 5400 3950 0    118  ~ 0
 BOARD 5-1
+Text Notes 3750 6800 0    50   ~ 0
+LAG OUT
 $EndSCHEMATC
