File: 4022 Noise/4022 Noise.sch (KiCad schematic (older format))
At the start: 18 parts, among them J2 GROUND, J5 OUTPUT, J6 POSITIVE SUPPLY, J7 GROUND, J8 NEGATIVE SUPPLY, Q1 2N5172

Commit message: fix value
Parts:
- C1: value 1.0 -> 1uF 35V
Changed lines of the file:
@@
 P 4650 3050
 F 0 "C1" V 4905 3050 50  0000 C CNN
-F 1 "1.0" V 4814 3050 50  0000 C CNN
+F 1 "1uF 35V" V 4814 3050 50  0000 C CNN
 F 2 "" H 4688 2900 50  0001 C CNN
 F 3 "~" H 4650 3050 50  0001 C CNN
