File: Board 4/Board 4.sch (KiCad schematic (older format))
At the start: 101 parts, among them Q6 2N5172, T60 output to left power amp, T65 output to right power amp

Commit message: Board 4 finalized
Parts:
- added A20: LM301, symbol Amplifier_Operational:LM301
- added C66: 30pF, symbol Device:C
- added C67: 50pF, symbol Device:C
- added C69: CP, symbol Device:CP
- added D21, D22, D23, D24, D25: 1N4148, Diode_THT:D_DO-35_SOD27_P7.62mm_Horizontal, symbol Diode:1N4148
- added E100, E45, E46, E47, E48: PJ301BM, symbol w_connector:PJ301BM
- added J100: VCA OUT, symbol Connector_Generic:Conn_01x01
- added Q5: 2N5460, symbol Device:Q_PJFET_SDG
- added R170: 2.2k, symbol Device:R
- added R171, R178, R199: 1k, symbol Device:R
- added R172: 68k, symbol Device:R
- added R173: 3.9k, symbol Device:R
- added R174, R175: 1M LOG, symbol Device:R_POT_TRIM
- added R176, R214: 10k, symbol Device:R
- added R177: 22k, symbol Device:R
- added SW1: manual start, symbol Switch:SW_Push
- added SW8: ~, symbol Switch:SW_DPDT_x2
- added T45: FROM ??? ??? BOARD 5-1, symbol Connector_Generic:Conn_01x01
- added T46: KEYBOARD GATE, symbol Connector_Generic:Conn_01x01
- added T47: TRIGGER, symbol Connector_Generic:Conn_01x01
- R183: value 9.1k 5% -> 9.1k 1%
- R184: value 10k 5% -> 10k 1%
- R205, R207: value 820k -> 820R
- gave numbers to parts that had none: 6
- renumbered E65 to E66, R195 to R193
Connections:
- net +15V: now also A20.7 (V+), R171.1
- net -15V: now also A20.4 (V-)
- net GND: now also C69.2, Q5.2 (D), R170.2, R173.2, R176.2
- net at BADSR-2.1 (Pin_1): now also D22.1 (K), D23.1 (K), R172.2, R214.2
- net at BADSR-1.1 (Pin_1): now also D21.1 (K), D24.1 (K)
- net at BVCA-5.1 (Pin_1): now also R199.2
- net at E52.2: now also E48.3, R178.2
- new net: A20.1 (BAL), C66.1
- new net: A20.2 (-), C67.2, R176.1, R177.2
- new net: A20.3 (+), C69.1, R174.3, R175.1, R175.2
- new net: A20.6, C67.1, R177.1, R178.1
- new net: A20.8 (C/B), C66.2
- new net: Q5.1 (S), R175.3
- new net: D25.1 (K), R174.1, R174.2
- new net: D25.2 (A), R172.1, R173.1
- new net: Q5.3 (G), R214.1
- new net: D22.2 (A), SW8.2 (B)
- new net: D23.2 (A), D24.2 (A), SW1.1
- new net: E45.3, SW8.1 (A), SW8.4 (A), T45.1 (Pin_1)
- new net: E46.3, SW8.3 (C), T46.1 (Pin_1)
- new net: D21.2 (A), SW8.5 (B)
- new net: E47.3, SW8.6 (C), T47.1 (Pin_1)
- new net: R170.1, R171.2, SW1.2
- new net: E100.3, J100.1 (Pin_1), R199.1
- no-connect marks 18 -> 29
Other:
- note added: "AR output"
- note added: "attack"
- note added: "doesn't have a number on the schematics"
- note added: "release"
- note added: "reverb output and right output has the same number: E65\nreverb output renamed to E66"
- note added: "sample and hold\nkbd gate switch"
- note added: "to right mixer input"

Commit message: Lots of fixes from patroche schematics/pcb
Parts:
- C69: value CP -> 1uF 35V
- R181: value 1M LOG -> 100k LIN
- R187, R188: value 100k LOG -> 100k LIN
Changed lines of the file:
@@
 P 11850 4700
 F 0 "R181" V 11735 4700 50  0000 C CNN
-F 1 "1M LOG" V 11644 4700 50  0000 C CNN
+F 1 "100k LIN" V 11644 4700 50  0000 C CNN
 F 2 "" H 11850 4700 50  0001 C CNN
 F 3 "~" H 11850 4700 50  0001 C CNN
@@
 P 10900 8750
 F 0 "R187" H 10830 8796 50  0000 R CNN
-F 1 "100k LOG" H 10830 8705 50  0000 R CNN
+F 1 "100k LIN" H 10830 8705 50  0000 R CNN
 F 2 "" H 10900 8750 50  0001 C CNN
 F 3 "~" H 10900 8750 50  0001 C CNN
@@
 P 11550 8750
 F 0 "R188" H 11480 8796 50  0000 R CNN
-F 1 "100k LOG" H 11480 8705 50  0000 R CNN
+F 1 "100k LIN" H 11480 8705 50  0000 R CNN
 F 2 "" H 11550 8750 50  0001 C CNN
 F 3 "~" H 11550 8750 50  0001 C CNN
@@
 P 5100 10000
 F 0 "C69" H 5218 10046 50  0000 L CNN
-F 1 "CP" H 5218 9955 50  0000 L CNN
+F 1 "1uF 35V" H 5218 9955 50  0000 L CNN
 F 2 "" H 5138 9850 50  0001 C CNN
 F 3 "~" H 5100 10000 50  0001 C CNN
