File: Board 5-1/Board 5-1.sch (KiCad schematic (older format))
At the start: 170 parts, among them J10 LAG OUT, J11 OUT, J12 OUT, J13 LAG IN/TIME, J18 S/H EXT CLOCK IN, J19 S/H OUTPUT, J20 S/H INPUT, J21 CLOCK OUT, J22 'B', J23 'C', J24 'A', J3 NOISE, J4 NOISE COLOR, J4015-1 S/H INPUT, J4015-4 S/H CLOCK IN, J4015-5 OUT, J4015-6 +15V, J4015-7 GND, J4015-8 -15V, J4022-2 GND, J4022-6 +15V, J4022-7 GND, J4022-8 -15V, J5 NOISE LEVEL, J6 NOISE OUT, Q30 D40D4, Q31 D40D4, Q32 D41D2, Q33 D41D2, Q34 2N5172, Q35 2N5172, Q36 2N5172, Q37 2N5172, Q38 2N5172, Q39 2N5172, Q40 2N4392, Q41 2N4392, Q43 2N6076, Q44 2N6076, Q45 2N4870

Commit message: board 5-1 fix values
Parts:
- C110, C113, C119, C120: value 0.001uF -> 1nF
- C116, C118: value 0.01uF -> 10nF
- C90: value 0.02uF -> 20nF
- C92: value 0.002uF -> 2nF
- R365: value 3.31k -> 3.3M
Changed lines of the file:
@@
 P 16800 13300
 F 0 "C119" V 16548 13300 50  0000 C CNN
-F 1 "0.001uF" V 16639 13300 50  0000 C CNN
+F 1 "1nF" V 16639 13300 50  0000 C CNN
 F 2 "" H 16838 13150 50  0001 C CNN
 F 3 "~" H 16800 13300 50  0001 C CNN
@@
 P 10250 14950
 F 0 "C116" H 10159 14904 50  0000 R CNN
-F 1 "0.01uF" H 10159 14995 50  0000 R CNN
+F 1 "10nF" H 10159 14995 50  0000 R CNN
 F 2 "" H 10250 14950 50  0001 C CNN
 F 3 "~" H 10250 14950 50  0001 C CNN
@@
 P 11650 14700
 F 0 "C118" H 11765 14746 50  0000 L CNN
-F 1 "0.01uF" H 11765 14655 50  0000 L CNN
+F 1 "10nF" H 11765 14655 50  0000 L CNN
 F 2 "" H 11688 14550 50  0001 C CNN
 F 3 "~" H 11650 14700 50  0001 C CNN
@@
 P 2550 2750
 F 0 "C92" V 2298 2750 50  0000 C CNN
-F 1 "0.002uF" V 2389 2750 50  0000 C CNN
+F 1 "2nF" V 2389 2750 50  0000 C CNN
 F 2 "" H 2588 2600 50  0001 C CNN
 F 3 "~" H 2550 2750 50  0001 C CNN
@@
 P 1400 2800
 F 0 "C90" H 1285 2754 50  0000 R CNN
-F 1 "0.02uF" H 1285 2845 50  0000 R CNN
+F 1 "20nF" H 1285 2845 50  0000 R CNN
 F 2 "" H 1438 2650 50  0001 C CNN
 F 3 "~" H 1400 2800 50  0001 C CNN
@@
 P 12200 9900
 F 0 "C113" H 12085 9854 50  0000 R CNN
-F 1 "0.001uF" H 12085 9945 50  0000 R CNN
+F 1 "1nF" H 12085 9945 50  0000 R CNN
 F 2 "" H 12238 9750 50  0001 C CNN
 F 3 "~" H 12200 9900 50  0001 C CNN
@@
 P 12500 8900
 F 0 "C120" V 12248 8900 50  0000 C CNN
-F 1 "0.001uF" V 12339 8900 50  0000 C CNN
+F 1 "1nF" V 12339 8900 50  0000 C CNN
 F 2 "" H 12538 8750 50  0001 C CNN
 F 3 "~" H 12500 8900 50  0001 C CNN
@@
 P 13300 8900
 F 0 "C110" V 13048 8900 50  0000 C CNN
-F 1 "0.001uF" V 13139 8900 50  0000 C CNN
+F 1 "1nF" V 13139 8900 50  0000 C CNN
 F 2 "" H 13338 8750 50  0001 C CNN
 F 3 "~" H 13300 8900 50  0001 C CNN
@@
 P 13850 9250
 F 0 "R365" V 13643 9250 50  0000 C CNN
-F 1 "3.31k" V 13734 9250 50  0000 C CNN
+F 1 "3.3M" V 13734 9250 50  0000 C CNN
 F 2 "" V 13780 9250 50  0001 C CNN
 F 3 "~" H 13850 9250 50  0001 C CNN

Commit message: Lots of fixes from patroche schematics/pcb
Parts:
- R345, R346, R355, R356: value 10R -> 10R 1/2W
- renumbered R364 to R369, R587 to R387
Connections:
- net -15V: now also Q36.1 (E)
- net at R359.1: now also Q36.3 (B), R358.2; no longer Q36.1 (E)
Other:
- note added: "C390 is named C123 which is duplicate, renamed\nsame for C128 which become C341\nQ45 (2N6076) -> Q43\nR363 -> R343\nR389 -> RV389\nR391 (int clock) -> R399\nR390 (int clock) -> R394\nC108 become C128"
- note removed: "C390 is named C123 which is duplicate, renamed\nsame for C128 which become C341\nQ45 (2N6076) -> Q43\nR363 -> R343\nR391 -> R399\nR389 -> RV389\nR391 (int clock) -> R394"
- moved on the sheet: Q36, R357, R358, R359
Changed lines of the file:
@@
 L Device:Q_NPN_ECB Q36
 U 1 1 613493F9
-P 11600 9250
-F 0 "Q36" H 11791 9296 50  0000 L CNN
-F 1 "2N5172" H 11791 9205 50  0000 L CNN
-F 2 "" H 11800 9350 50  0001 C CNN
-F 3 "~" H 11600 9250 50  0001 C CNN
-	1    11600 9250
+P 11450 9250
+F 0 "Q36" H 11641 9296 50  0000 L CNN
+F 1 "2N5172" H 11641 9205 50  0000 L CNN
+F 2 "" H 11650 9350 50  0001 C CNN
+F 3 "~" H 11450 9250 50  0001 C CNN
+	1    11450 9250
 	-1   0    0    -1
 $EndComp
@@
 P 20600 2050
 F 0 "R345" H 20670 2096 50  0000 L CNN
-F 1 "10R" H 20670 2005 50  0000 L CNN
+F 1 "10R 1/2W" H 20670 2005 50  0000 L CNN
 F 2 "" V 20530 2050 50  0001 C CNN
 F 3 "~" H 20600 2050 50  0001 C CNN
@@
 P 20600 2350
 F 0 "R346" H 20670 2396 50  0000 L CNN
-F 1 "10R" H 20670 2305 50  0000 L CNN
+F 1 "10R 1/2W" H 20670 2305 50  0000 L CNN
 F 2 "" V 20530 2350 50  0001 C CNN
 F 3 "~" H 20600 2350 50  0001 C CNN
@@
 P 20600 4950
 F 0 "R355" H 20670 4996 50  0000 L CNN
-F 1 "10R" H 20670 4905 50  0000 L CNN
+F 1 "10R 1/2W" H 20670 4905 50  0000 L CNN
 F 2 "" V 20530 4950 50  0001 C CNN
 F 3 "~" H 20600 4950 50  0001 C CNN
@@
 P 20600 5250
 F 0 "R356" H 20670 5296 50  0000 L CNN
-F 1 "10R" H 20670 5205 50  0000 L CNN
+F 1 "10R 1/2W" H 20670 5205 50  0000 L CNN
 F 2 "" V 20530 5250 50  0001 C CNN
 F 3 "~" H 20600 5250 50  0001 C CNN
@@
 	11650 14950 11600 14950
 $Comp
-L Device:R R587
+L Device:R R387
 U 1 1 6141F871
 P 11250 14400
-F 0 "R587" H 11320 14446 50  0000 L CNN
+F 0 "R387" H 11320 14446 50  0000 L CNN
 F 1 "4.7k" H 11320 14355 50  0000 L CNN
 F 2 "" V 11180 14400 50  0001 C CNN
@@
 L Device:R R357
 U 1 1 61D10D63
-P 11500 8850
-F 0 "R357" H 11570 8896 50  0000 L CNN
-F 1 "22M" H 11570 8805 50  0000 L CNN
-F 2 "" V 11430 8850 50  0001 C CNN
-F 3 "~" H 11500 8850 50  0001 C CNN
-	1    11500 8850
+P 11350 8850
+F 0 "R357" H 11420 8896 50  0000 L CNN
+F 1 "22M" H 11420 8805 50  0000 L CNN
+F 2 "" V 11280 8850 50  0001 C CNN
+F 3 "~" H 11350 8850 50  0001 C CNN
+	1    11350 8850
 	1    0    0    -1
 $EndComp
 Wire Wire Line
-	11500 9000 11500 9050
+	11350 9000 11350 9050
 $Comp
 L power:+15V #PWR0154
 U 1 1 61D29F9A
-P 11500 8650
-F 0 "#PWR0154" H 11500 8500 50  0001 C CNN
-F 1 "+15V" H 11515 8823 50  0000 C CNN
-F 2 "" H 11500 8650 50  0001 C CNN
-F 3 "" H 11500 8650 50  0001 C CNN
-	1    11500 8650
+P 11350 8650
+F 0 "#PWR0154" H 11350 8500 50  0001 C CNN
+F 1 "+15V" H 11365 8823 50  0000 C CNN
+F 2 "" H 11350 8650 50  0001 C CNN
+F 3 "" H 11350 8650 50  0001 C CNN
+	1    11350 8650
 	1    0    0    -1
 $EndComp
 Wire Wire Line
-	11500 8650 11500 8700
+	11350 8650 11350 8700
 $Comp
 L Device:R R359
 U 1 1 61D5A820
-P 11500 9650
-F 0 "R359" H 11570 9696 50  0000 L CNN
-F 1 "100k" H 11570 9605 50  0000 L CNN
-F 2 "" V 11430 9650 50  0001 C CNN
-F 3 "~" H 11500 9650 50  0001 C CNN
-	1    11500 9650
-	1    0    0    -1
+P 11650 9650
+F 0 "R359" H 11720 9696 50  0000 L CNN
+F 1 "100k" H 11720 9605 50  0000 L CNN
+F 2 "" V 11580 9650 50  0001 C CNN
+F 3 "~" H 11650 9650 50  0001 C CNN
+	1    11650 9650
+	-1   0    0    -1
 $EndComp
-Wire Wire Line
-	11500 9500 11500 9450
 $Comp
 L power:-15V #PWR0155
 U 1 1 61D73F8F
-P 11500 9850
-F 0 "#PWR0155" H 11500 9950 50  0001 C CNN
-F 1 "-15V" H 11515 10023 50  0000 C CNN
-F 2 "" H 11500 9850 50  0001 C CNN
-F 3 "" H 11500 9850 50  0001 C CNN
-	1    11500 9850
+P 11650 9850
+F 0 "#PWR0155" H 11650 9950 50  0001 C CNN
+F 1 "-15V" H 11665 10023 50  0000 C CNN
+F 2 "" H 11650 9850 50  0001 C CNN
+F 3 "" H 11650 9850 50  0001 C CNN
+	1    11650 9850
 	-1   0    0    1
 $EndComp
 Wire Wire Line
-	11500 9850 11500 9800
+	11650 9850 11650 9800
 $Comp
 L Device:R R358
 U 1 1 61DA55C2
-P 12000 9250
-F 0 "R358" V 11793 9250 50  0000 C CNN
-F 1 "3.3M" V 11884 9250 50  0000 C CNN
-F 2 "" V 11930 9250 50  0001 C CNN
-F 3 "~" H 12000 9250 50  0001 C CNN
-	1    12000 9250
+P 11900 9250
+F 0 "R358" V 11693 9250 50  0000 C CNN
+F 1 "3.3M" V 11784 9250 50  0000 C CNN
+F 2 "" V 11830 9250 50  0001 C CNN
+F 3 "~" H 11900 9250 50  0001 C CNN
+	1    11900 9250
 	0    1    1    0
 $EndComp
 Wire Wire Line
-	11850 9250 11800 9250
+	11750 9250 11650 9250
 $Comp
 L Device:C C113
@@
 Connection ~ 12200 9250
 Wire Wire Line
-	12150 9250 12200 9250
+	12050 9250 12200 9250
 Wire Wire Line
 	12200 9700 12200 9650
@@
 Wire Wire Line
 	14000 9250 14100 9250
-$Comp
-L Device:R R364
-U 1 1 62290171
-P 14100 9600
-F 0 "R364" H 14030 9554 50  0000 R CNN
-F 1 "100k" H 14030 9645 50  0000 R CNN
-F 2 "" V 14030 9600 50  0001 C CNN
-F 3 "~" H 14100 9600 50  0001 C CNN
-	1    14100 9600
-	-1   0    0    1
-$EndComp
 Wire Wire Line
 	14100 9750 14450 9750
@@
 $EndComp
 Wire Wire Line
-	11500 9000 11800 9000
+	11350 9000 11800 9000
 Wire Wire Line
 	11800 9000 11800 7450
 Wire Wire Line
 	11800 7450 15800 7450
-Connection ~ 11500 9000
+Connection ~ 11350 9000
 Connection ~ 15800 7450
 Wire Wire Line
@@
 Connection ~ 9500 13400
 Text Notes 18700 15350 0    50   ~ 0
-C390 is named C123 which is duplicate, renamed\nsame for C128 which become C341\nQ45 (2N6076) -> Q43\nR363 -> R343\nR391 -> R399\nR389 -> RV389\nR391 (int clock) -> R394
+C390 is named C123 which is duplicate, renamed\nsame for C128 which become C341\nQ45 (2N6076) -> Q43\nR363 -> R343\nR389 -> RV389\nR391 (int clock) -> R399\nR390 (int clock) -> R394\nC108 become C128
 $Comp
 L power:GND #PWR0175
@@
 	0    -1   -1   0
 $EndComp
+Connection ~ 11650 9250
+Wire Wire Line
+	11350 9800 11650 9800
+Wire Wire Line
+	11350 9450 11350 9800
+Connection ~ 11650 9800
+Wire Wire Line
+	11650 9250 11650 9500
+$Comp
+L Device:R R369
+U 1 1 62290171
+P 14100 9600
+F 0 "R369" H 14030 9554 50  0000 R CNN
+F 1 "100k" H 14030 9645 50  0000 R CNN
+F 2 "" V 14030 9600 50  0001 C CNN
+F 3 "~" H 14100 9600 50  0001 C CNN
+	1    14100 9600
+	-1   0    0    1
+$EndComp
 $EndSCHEMATC
