File: 4015 Sample and Hold/4015 Sample and Hold.sch (KiCad schematic (older format))
At the start: 46 parts, among them J1 INPUT, J4 SAMPLE IN, J5 OUTPUT, J6 POSITIVE SUPPLY, J7 GROUND, J8 NEGATIVE SUPPLY, Q1 2N5172, Q2 2N3906, Q3 2N5172, Q4 BF245A or 2SK30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

Commit message: fixes
Parts:
- A1, A2: value LM301 -> LM301A
- C1, C2, C3, C4, C5, C6, C7: notes (none) -> ceramic
- C8: value 0.022uF polycarbonate -> 22nF polycarbonate; notes (none) -> polycarbonate
- Q7-1, Q7-2: notes (none) -> they have to be matched and thermal paired
Changed lines of the file:
@@
 F 2 "" H 1338 1250 50  0001 C CNN
 F 3 "~" H 1300 1400 50  0001 C CNN
+F 4 "ceramic" H 1300 1400 50  0001 C CNN "notes"
 	1    1300 1400
 	1    0    0    -1
@@
 F 2 "" H 1338 1650 50  0001 C CNN
 F 3 "~" H 1300 1800 50  0001 C CNN
+F 4 "ceramic" H 1300 1800 50  0001 C CNN "notes"
 	1    1300 1800
 	1    0    0    -1
@@
 P 9050 2600
 F 0 "A2" H 9394 2646 50  0000 L CNN
-F 1 "LM301" H 9394 2555 50  0000 L CNN
+F 1 "LM301A" H 9394 2555 50  0000 L CNN
 F 2 "" H 9100 2650 50  0001 C CNN
 F 3 "http://www.ti.com/lit/ds/symlink/lm101a-n.pdf" H 9100 2750 50  0001 C CNN
@@
 F 2 "Package_TO_SOT_THT:TO-92_Inline" H 7050 2325 50  0001 L CIN
 F 3 "https://www.onsemi.com/pub/Collateral/BF245A-D.PDF" H 6850 2400 50  0001 L CNN
+F 4 "they have to be matched and thermal paired" H 6850 2400 50  0001 C CNN "notes"
 	1    6850 2400
 	1    0    0    -1
@@
 F 2 "Package_TO_SOT_THT:TO-92_Inline" H 7050 3025 50  0001 L CIN
 F 3 "https://www.onsemi.com/pub/Collateral/BF245A-D.PDF" H 6850 3100 50  0001 L CNN
+F 4 "they have to be matched and thermal paired" H 6850 3100 50  0001 C CNN "notes"
 	1    6850 3100
 	1    0    0    1
@@
 F 2 "" H 2538 3200 50  0001 C CNN
 F 3 "~" H 2500 3350 50  0001 C CNN
+F 4 "ceramic" H 2500 3350 50  0001 C CNN "notes"
 	1    2500 3350
 	1    0    0    -1
@@
 F 2 "" H 3388 3050 50  0001 C CNN
 F 3 "~" H 3350 3200 50  0001 C CNN
+F 4 "ceramic" H 3350 3200 50  0001 C CNN "notes"
 	1    3350 3200
 	0    1    1    0
@@
 P 3150 3650
 F 0 "A1" H 3494 3696 50  0000 L CNN
-F 1 "LM301" H 3494 3605 50  0000 L CNN
+F 1 "LM301A" H 3494 3605 50  0000 L CNN
 F 2 "" H 3200 3700 50  0001 C CNN
 F 3 "http://www.ti.com/lit/ds/symlink/lm101a-n.pdf" H 3200 3800 50  0001 C CNN
@@
 F 2 "" H 2788 4400 50  0001 C CNN
 F 3 "~" H 2750 4550 50  0001 C CNN
+F 4 "ceramic" H 2750 4550 50  0001 C CNN "notes"
 	1    2750 4550
 	0    1    1    0
@@
 P 6300 3850
 F 0 "C8" V 6048 3850 50  0000 C CNN
-F 1 "0.022uF polycarbonate" V 6450 4200 50  0000 C CNN
+F 1 "22nF polycarbonate" V 6450 4200 50  0000 C CNN
 F 2 "" H 6338 3700 50  0001 C CNN
 F 3 "~" H 6300 3850 50  0001 C CNN
+F 4 "polycarbonate" H 6300 3850 50  0001 C CNN "notes"
 	1    6300 3850
 	0    1    1    0
@@
 F 2 "" H 8338 1850 50  0001 C CNN
 F 3 "~" H 8300 2000 50  0001 C CNN
+F 4 "ceramic" H 8300 2000 50  0001 C CNN "notes"
 	1    8300 2000
 	0    1    1    0
@@
 F 2 "" H 9388 2150 50  0001 C CNN
 F 3 "~" H 9350 2300 50  0001 C CNN
+F 4 "ceramic" H 9350 2300 50  0001 C CNN "notes"
 	1    9350 2300
 	0    -1   -1   0

Commit message: Fix value in 4015
Parts:
- C3: value 20nF -> 20pF
Changed lines of the file:
@@
 P 2500 3350
 F 0 "C3" H 2615 3396 50  0000 L CNN
-F 1 "20nF" H 2615 3305 50  0000 L CNN
+F 1 "20pF" H 2615 3305 50  0000 L CNN
 F 2 "" H 2538 3200 50  0001 C CNN
 F 3 "~" H 2500 3350 50  0001 C CNN

Commit message: various fixes
Other:
- note added: "thermal pair"
- note removed: "match and thermal pair"
Changed lines of the file:
@@
 Wire Wire Line
 	8400 3400 8400 2500
-Text Notes 7350 2350 0    50   ~ 0
-match and thermal pair
+Text Notes 7600 2350 0    50   ~ 0
+thermal pair
 Wire Notes Line
-	7300 2250 8300 2250
+	7550 2250 8100 2250
 Wire Notes Line
-	8300 2250 8300 2400
+	8100 2250 8100 2400
 Wire Notes Line
-	8300 2400 7300 2400
+	8100 2400 7550 2400
 Wire Notes Line
-	7300 2400 7300 2250
+	7550 2400 7550 2250
 $EndSCHEMATC
