File: 4019 VCA/4019 VCA.sch (KiCad schematic (older format))
At the start: 66 parts, among them J1 AUDIO +, J10 LINEAR GAIN, J11 HIGH FREQ. REJECT, J14 LINEAR GAIN, J18 EXPONENTIAL GAIN, J19 REJECTION CONTROL, J2 AUDIO -, J3 LINEAR INPUT, J4 INPUT, J5 OUTPUT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

Commit message: various fixes
Other:
- note added: "match and thermal pair"
Changed lines of the file:
@@
 Wire Wire Line
 	8600 4650 8750 4650
+Text Notes 6300 1800 0    79   ~ 0
+match and thermal pair
+Wire Notes Line
+	6250 1650 7800 1650
+Wire Notes Line
+	7800 1650 7800 1850
+Wire Notes Line
+	7800 1850 6250 1850
+Wire Notes Line
+	6250 1850 6250 1650
 $EndSCHEMATC

Commit message: various fixes
Other:
- note added: "thermal pair"
Changed lines of the file:
@@
 Wire Wire Line
 	8600 4650 8750 4650
-Text Notes 6300 1800 0    79   ~ 0
+Text Notes 6150 2800 0    79   ~ 0
 match and thermal pair
-Wire Notes Line
-	6250 1650 7800 1650
-Wire Notes Line
-	7800 1650 7800 1850
-Wire Notes Line
-	7800 1850 6250 1850
-Wire Notes Line
-	6250 1850 6250 1650
+Text Notes 6150 5850 0    79   ~ 0
+match and thermal pair
+Text Notes 3300 3300 0    79   ~ 0
+thermal pair
+Text Notes 3600 1550 0    79   ~ 0
+match and thermal pair
 $EndSCHEMATC
