File: 4027 VCO/4027 VCO.sch (KiCad schematic (older format))
At the start: 43 parts, among them J18 L.F. CAP, J19 TRIM INPUT, J2 CONT. INPUT, J5 SAW. OUT, J6 POSITIVE SUPPLY, J7 GROUND, J8 NEGATIVE SUPPLY, Q1 2N3906, Q2 2N3904, Q3 2N5459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

Commit message: various fixes
Changed lines of the file:
@@
+	1    0    0    -1
+$EndComp
+$Comp
+L power:PWR_FLAG #FLG?
+U 1 1 60B56473
+P 1150 2000
+F 0 "#FLG?" H 1150 2075 50  0001 C CNN
+F 1 "PWR_FLAG" H 1050 2150 50  0000 L CNN
+F 2 "" H 1150 2000 50  0001 C CNN
+F 3 "~" H 1150 2000 50  0001 C CNN
+	1    1150 2000
 	1    0    0    -1
 $EndComp

Commit message: Lots of fixes from patroche schematics/pcb
Parts:
- R4: value 1.84k 1% -> 1.87k - tempco - 3500ppm 1w 3%; Notes 1.87k 3% ? -> 1.87k - tempco - 3500ppm 1w 3%
Changed lines of the file:
@@
 U 1 1 60270901
 P 3500 4200
-F 0 "R4" H 3430 4154 50  0000 R CNN
-F 1 "1.84k 1%" H 3430 4245 50  0000 R CNN
+F 0 "R4" H 3650 4350 50  0000 R CNN
+F 1 "1.87k - tempco - 3500ppm 1w 3%" H 3600 4650 50  0000 R CNN
 F 2 "" V 3430 4200 50  0001 C CNN
 F 3 "~" H 3500 4200 50  0001 C CNN
-F 4 "1.87k 3% ?" H 3500 4200 50  0001 C CNN "Notes"
+F 4 "1.87k - tempco - 3500ppm 1w 3%" H 3500 4200 50  0001 C CNN "Notes"
 	1    3500 4200
 	-1   0    0    1

Commit message: various fixes
Other:
- note added: "thermal pair"
- note removed: "match and thermal pair"
Changed lines of the file:
@@
 	3650 3850 3650 4150
 Text Notes 3750 1050 0    50   ~ 0
-match and thermal pair
+thermal pair
 Wire Notes Line
-	3700 950  4700 950
+	3700 950  4250 950
 Wire Notes Line
-	4700 950  4700 1100
+	4250 950  4250 1100
 Wire Notes Line
-	4700 1100 3700 1100
+	4250 1100 3700 1100
 Wire Notes Line
 	3700 1100 3700 950
