File: 4072 VCF/4072 VCF.sch (KiCad schematic (older format))
At the start: 85 parts, among them J1 NON-INVERTING INPUT, J10 GAIN TRIM, J14 CVR TRIM, J18 CVR TRIM, J2 INVERTING INPUT, J3 Fc CONTROL INPUT, J5 OUTPUT, J6 POSITIVE SUPPLY, J7 GROUND, J8 NEGATIVE SUPPLY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

Commit message: various fixes
Changed lines of the file:
@@
 Text Notes 8600 3800 0    39   ~ 0
 apparently this caps was added\nin the 4072 from the 4072 edit
+$Comp
+L power:PWR_FLAG #FLG?
+U 1 1 60B4E714
+P 2800 7650
+F 0 "#FLG?" H 2800 7725 50  0001 C CNN
+F 1 "PWR_FLAG" V 2800 7778 50  0000 L CNN
+F 2 "" H 2800 7650 50  0001 C CNN
+F 3 "~" H 2800 7650 50  0001 C CNN
+	1    2800 7650
+	0    1    1    0
+$EndComp
 $EndSCHEMATC

Commit message: various fixes
Other:
- note added: "thermal pair"
- note removed: "match and thermal pair"
Changed lines of the file:
@@
 	13850 7000 13850 6450
 Connection ~ 13850 6450
-Text Notes 9700 3550 0    79   ~ 0
-match and thermal pair
+Text Notes 10250 3500 0    79   ~ 0
+thermal pair
 Wire Notes Line
-	9650 3400 9650 3600
+	10200 3350 10200 3550
 Wire Notes Line
-	9650 3600 11200 3600
+	10200 3550 11050 3550
 Wire Notes Line
-	11200 3600 11200 3400
+	11050 3550 11050 3350
 Wire Notes Line
-	11200 3400 9650 3400
+	11050 3350 10200 3350
 Text Notes 3800 2000 0    79   ~ 0
 Exponential Converter
