File: Board 2-1/Board 2-1.sch (KiCad schematic (older format))
At the start: 48 parts, among them J1 FROM PULSE WIDTH SLIDER, J2 SAWTOOTH FROM VCO-2, J3 PULSE WAVE OUTPUT, J4 POSITIVE SUPPLY, J5 GND, J6 NEGATIVE SUPPLY, J7 PULSE WIDTH MOD IN, J8 SINE WAVE OUTPUT, J9 TRIANGLE WAVE OUT, Q1 2N3906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

Commit message: Lots of fixes from patroche schematics/pcb
Parts:
- added R124: 68k, symbol Device:R
- added R125: 100k, symbol Device:R_POT_TRIM
Connections:
- net +15V: now also R125.1
- net GND: now also R125.3
- net at A16.2 (-), C56.2, R121.2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: now also R124.1
- new net: R124.2, R125.2
Other:
- note added: "DC OFFSET"
Changed lines of the file:
@@
 Wire Wire Line
 	2200 1900 2200 5750
+$Comp
+L Device:R R124
+U 1 1 62E2B559
+P 7000 5750
+F 0 "R124" V 7207 5750 50  0000 C CNN
+F 1 "68k" V 7116 5750 50  0000 C CNN
+F 2 "" V 6930 5750 50  0001 C CNN
+F 3 "~" H 7000 5750 50  0001 C CNN
+	1    7000 5750
+	1    0    0    -1
+$EndComp
+Wire Wire Line
+	7000 5600 7000 5450
+$Comp
+L Device:R_POT_TRIM R125
+U 1 1 62E310F9
+P 7000 6050
+F 0 "R125" V 6885 6050 50  0000 C CNN
+F 1 "100k" V 6794 6050 50  0000 C CNN
+F 2 "" H 7000 6050 50  0001 C CNN
+F 3 "~" H 7000 6050 50  0001 C CNN
+	1    7000 6050
+	0    -1   -1   0
+$EndComp
+$Comp
+L power:+15V #PWR?
+U 1 1 62E319ED
+P 6850 6050
+F 0 "#PWR?" H 6850 5900 50  0001 C CNN
+F 1 "+15V" H 6865 6223 50  0000 C CNN
+F 2 "" H 6850 6050 50  0001 C CNN
+F 3 "" H 6850 6050 50  0001 C CNN
+	1    6850 6050
+	0    -1   -1   0
+$EndComp
+$Comp
+L power:GND #PWR?
+U 1 1 62E321C7
+P 7150 6050
+F 0 "#PWR?" H 7150 5800 50  0001 C CNN
+F 1 "GND" H 7155 5877 50  0000 C CNN
+F 2 "" H 7150 6050 50  0001 C CNN
+F 3 "" H 7150 6050 50  0001 C CNN
+	1    7150 6050
+	0    -1   -1   0
+$EndComp
+Text Notes 6750 6400 0    50   ~ 0
+DC OFFSET
 $EndSCHEMATC

Commit message: various fixes
Other:
- note added: "thermal pair"
- note removed: "match and thermal pair"
Changed lines of the file:
@@
 	6900 1900 6900 1950
 Text Notes 6350 1200 0    50   ~ 0
-match and thermal pair
+thermal pair
 Wire Notes Line
-	6300 1100 7300 1100
+	6300 1100 6850 1100
 Wire Notes Line
-	7300 1100 7300 1250
+	6850 1100 6850 1250
 Wire Notes Line
-	7300 1250 6300 1250
+	6850 1250 6300 1250
 Wire Notes Line
 	6300 1250 6300 1100
